File: pcb/mantis.kicad_pcb (KiCad board)
At the start: 2 copper layers, 242 x 129.5 mm, 82 parts

Commit message: Mantis v0.2 PCBs
PCBs for Mantis v0.2 ready for manufacturing. The two PCBs are connected
with 2.54mm pitch headers. Optional M2 standoffs can de used to adjust
the height or provide more mechanical stability if needed.

The bottom PCB can be used to build a flat keyboard without the top PCB.

Signed-off-by: Felix Kuehling <felix.kuehling@gmail.com>
Parts:
- added ?: PinHeader_1x02_P2.54mm_Vertical, Connector_PinHeader_2.54mm:PinHeader_1x02_P2.54mm_Vertical, F.Cu at (84.5, 108.0)
- added ?: MountingHole_2.2mm_M2_Pad, MountingHole:MountingHole_2.2mm_M2_Pad, F.Cu at (130.2, 103.5)
- added ?: MountingHole_2.2mm_M2_Pad, MountingHole:MountingHole_2.2mm_M2_Pad, F.Cu at (86.4, 128.9)
- added ?: PinHeader_1x02_P2.54mm_Vertical, Connector_PinHeader_2.54mm:PinHeader_1x02_P2.54mm_Vertical, F.Cu at (106.0, 66.7)
- added ?: MountingHole_2.2mm_M2_Pad, MountingHole:MountingHole_2.2mm_M2_Pad, F.Cu at (162.6, 64.8)
- added ?: PinHeader_1x05_P2.54mm_Vertical, Connector_PinHeader_2.54mm:PinHeader_1x05_P2.54mm_Vertical, F.Cu at (130.2, 88.3)
- added ?: MountingHole_2.2mm_M2_Pad, MountingHole:MountingHole_2.2mm_M2_Pad, F.Cu at (98.4, 64.8)
- added ?: PinHeader_1x02_P2.54mm_Vertical, Connector_PinHeader_2.54mm:PinHeader_1x02_P2.54mm_Vertical, F.Cu at (152.4, 66.7)
- added ?: MountingHole_2.2mm_M2_Pad, MountingHole:MountingHole_2.2mm_M2_Pad, F.Cu at (175.3, 128.9)
- added ?: PinHeader_1x02_P2.54mm_Vertical, Connector_PinHeader_2.54mm:PinHeader_1x02_P2.54mm_Vertical, F.Cu at (174.0, 108.0)
- moved S9 78.0 mm to (75.2, 36.5)
- moved S29 77.9 mm to (185.8, 36.5)
- moved D9 77.1 mm to (83.8, 37.5)
- moved D29 76.9 mm to (194.2, 37.5)
- moved D16 66.4 mm to (73.0, 94.1)
- moved S16 65.4 mm to (64.5, 93.1)
- moved D36 50.3 mm to (205.0, 94.1)
- moved S36 49.9 mm to (196.5, 93.1)
- moved D24 49.7 mm to (215.8, 75.5)
- moved S24 48.6 mm to (207.2, 74.5)
- moved D17 46.4 mm to (83.8, 116.2)
- moved S17 46.3 mm to (75.2, 115.2)
- moved D34 46.2 mm to (151.2, 75.1)
- moved S34 46.1 mm to (142.8, 74.1)
- moved D19 43.2 mm to (116.0, 134.8)
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Connections:
- net index_r1 renamed c5_r2
- net index_r2 renamed c5_r3
- net index_r3 renamed c1_rt
- net inner_r1 renamed c3_rt
- net inner_r2 renamed c4_rt
- net inner_thumb renamed c2_rt
- net middle_r3 renamed c4_r3
- net mirror_index_r2 renamed c5m_r3
- net mirror_inner_r3 renamed c5m_rt
- net mirror_middle_r2 renamed c4m_r2
- net mirror_pinky_r2 renamed c1m_r3
- net mirror_pinky_r3 renamed c2m_r1
- net mirror_ring_r1 renamed c2m_r3
- net pinky_r1 renamed c1_r2
- net pinky_r3 renamed c2_r1
- net pinky_thumb renamed c1_r1
- net ring_thumb renamed c2_r2
- D1 pad 1: P3 -> P2
- D10 pad 2: P2 -> c4_r1
- D11 pad 1: middle_r2 -> P0
- D11 pad 2: middle_r2 -> c4_r2
- D13 pad 1: P3 -> P2
- D13 pad 2: P3 -> c5_r1
- D14 pad 1: P2 -> P0
- D15 pad 1: P0 -> P1
- D16 pad 1: P1 -> P3
- D18 pad 1: P2 -> P3
- D19 pad 1: P0 -> P3
- D2 pad 1: P2 -> P0
- D20 pad 1: P1 -> P3
- D20 pad 2: P1 -> c5_rt
- D21 pad 1: P3 -> P2
- D21 pad 2: P3 -> c1m_r1
- D22 pad 1: P2 -> P0
- D22 pad 2: P2 -> c1m_r2
- D23 pad 1: P0 -> P1
- D24 pad 1: P1 -> P2
- D25 pad 1: P3 -> P0
- D25 pad 2: P3 -> c2m_r2
- D26 pad 1: P2 -> P1
- D27 pad 1: mirror_ring_r2 -> P2
- D27 pad 2: mirror_ring_r2 -> c3m_r1
- D28 pad 1: P1 -> P0
- D28 pad 2: P1 -> c3m_r2
- D29 pad 1: P3 -> P1
- D29 pad 2: P3 -> c3m_r3
- D3 pad 1: P0 -> P1
- D3 pad 2: P0 -> c1_r3
- D30 pad 2: P2 -> c4m_r1
- D32 pad 1: mirror_middle_r3 -> P1
- D32 pad 2: P1 -> c4m_r3
- D33 pad 1: P3 -> P2
- D33 pad 2: P3 -> c5m_r1
- D34 pad 1: P2 -> P0
- D34 pad 2: P2 -> c5m_r2
- D35 pad 1: P0 -> P1
- D36 pad 1: P1 -> P3
- D36 pad 2: P1 -> c1m_rt
- D37 pad 2: P3 -> c2m_rt
- D38 pad 1: P2 -> P3
- D38 pad 2: P2 -> c3m_rt
- D39 pad 1: P0 -> P3
- D39 pad 2: P0 -> c4m_rt
- D4 pad 1: P1 -> P2
- D40 pad 1: P1 -> P3
- D5 pad 1: P3 -> P0
- D6 pad 1: P2 -> P1
- D6 pad 2: P2 -> c2_r3
- D7 pad 1: ring_r2 -> P2
- D7 pad 2: ring_r2 -> c3_r1
- D8 pad 1: P1 -> P0
- D8 pad 2: P1 -> c3_r2
- D9 pad 1: P3 -> P1
- D9 pad 2: P3 -> c3_r3
- S10 pad 1: middle_r1 -> c4_r1
- S10 pad 2: P15 -> P14
- S11 pad 1: middle_r2 -> c4_r2
- S11 pad 2: P15 -> P14
- S12 pad 2: P15 -> P14
- S13 pad 1: index_thumb -> c5_r1
- S13 pad 2: P14 -> P16
- S14 pad 2: P14 -> P16
- S15 pad 2: P14 -> P16
- S16 pad 2: P14 -> P19
- S17 pad 2: P16 -> P18
- S18 pad 2: P16 -> P15
- S19 pad 2: P16 -> P14
- S20 pad 1: inner_r3 -> c5_rt
- S21 pad 1: mirror_pinky_thumb -> c1m_r1
- S22 pad 1: mirror_pinky_r1 -> c1m_r2
- S24 pad 2: P4 -> P5
- S25 pad 1: mirror_ring_thumb -> c2m_r2
- S27 pad 1: mirror_ring_r2 -> c3m_r1
- S27 pad 2: P5 -> P6
- S28 pad 1: mirror_ring_r3 -> c3m_r2
- S28 pad 2: P5 -> P6
- S29 pad 1: mirror_middle_thumb -> c3m_r3
- S3 pad 1: pinky_r2 -> c1_r3
- S30 pad 1: mirror_middle_r1 -> c4m_r1
- S30 pad 2: P6 -> P7
- S31 pad 2: P6 -> P7
- S32 pad 1: mirror_middle_r3 -> c4m_r3
- S32 pad 2: P6 -> P7
- S33 pad 1: mirror_index_thumb -> c5m_r1
- S33 pad 2: P7 -> P8
- S34 pad 1: mirror_index_r1 -> c5m_r2
- S34 pad 2: P7 -> P8
- S35 pad 2: P7 -> P8
- S36 pad 1: mirror_index_r3 -> c1m_rt
- S36 pad 2: P7 -> P4
- S37 pad 1: mirror_inner_thumb -> c2m_rt
- S37 pad 2: P8 -> P5
- S38 pad 1: mirror_inner_r1 -> c3m_rt
- S38 pad 2: P8 -> P6
- S39 pad 1: mirror_inner_r2 -> c4m_rt
- S39 pad 2: P8 -> P7
- S4 pad 2: P19 -> P18
- S6 pad 1: ring_r1 -> c2_r3
- S7 pad 1: ring_r2 -> c3_r1
- S7 pad 2: P18 -> P15
- S8 pad 1: ring_r3 -> c3_r2
- S8 pad 2: P18 -> P15
- S9 pad 1: middle_thumb -> c3_r3
Routing:
- net P14: track 99.6 -> 183.4 mm
- net P18: track 134.8 -> 215.7 mm
- net P3: track 391.5 -> 318.3 mm
- net P5: track 117.4 -> 177.6 mm
- net P2: track 396.8 -> 342.6 mm
- net P7: track 79.3 -> 133.5 mm
- net P0: track 388.4 -> 335.8 mm
- net P6: track 111.6 -> 160.2 mm
- net P15: track 128.0 -> 171.0 mm
- net P4: track 155.2 -> 183.9 mm
- net P19: track 179.8 -> 198.1 mm
- net P1: track 328.5 -> 342.4 mm
- net mirror_pinky_thumb: track 10.9 -> 0.00 mm
- net mirror_middle_r1: track 10.9 -> 0.00 mm
- net inner_r3: track 10.9 -> 0.00 mm
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Other:
- board size 242 x 129.5 mm -> 220 x 129.3 mm
- board text added: "Mantis v0.2 Felix Kühling March 2023"
- board text removed: "Graphic: {dblquote}Praying mantis{dblquote} by HolleyandChris is licensed under CC BY 2.0. https://wordpress.org/openverse/image/ 07787e94-05c0-4aa9-a530-9cb8ce2a4666 Modified and converted to B/W SVG with Gimp and Inkscape by Felix Kühling"
- board text removed: "Mantis v0.1 Felix Kühling"
